File: Hokuto.kicad_sch (KiCad schematic)
At the start: 0 parts

Commit message: pcb mostly finished
Parts:
- added SW1, SW2, SW3, SW4, SW5, SW6: SW_Push, Button_Switch_Keyboard:SW_Cherry_MX_1.00u_PCB, symbol Switch:SW_Push
- added U1: XIAO-RP2040-DIP, Seeed Studio XIAO Series Library:XIAO-RP2040-DIP, symbol Seeed_Studio_XIAO_Series:XIAO-RP2040-DIP
Connections:
- new net GND: SW1.1, SW2.1, SW3.1, SW4.1, SW5.1, SW6.1, U1.13 (GND)
- new net SW1: SW1.2, U1.8 (GPIO1/RX)
- new net SW2: SW2.2, U1.9 (GPIO2/SCK)
- new net SW3: SW3.2, U1.10 (GPIO4/MISO)
- new net SW4: SW4.2, U1.11 (GPIO3/MOSI)
- new net SW5: SW5.2, U1.7 (GPIO0/TX)
- new net SW6: SW6.2, U1.6 (GPIO7/SCL)
- new net SW7: U1.5 (GPIO6/SDA)
- new net SW8: U1.4 (GPIO29/ADC3/A3)
- new net SW9: U1.3 (GPIO28/ADC2/A2)
